File: hardware/RF_Board/RF_Board.kicad_sch (KiCad schematic)
At the start: 59 parts, among them U1 MSP430FR2355TPT, U10 QPL9096, U11 QPL9096, U12 74AHC04, U2 MSP430FR2355TPT, U3 CC2500, U4 HMC574, U5 HMC574, U6 YAT-5A+, U7 SKY65900-11, U8 LFCN-2750+, U9 DEA202450BT-1213C1, Y1 Crystal_GND24

Commit message: more RF board schematic work
Parts:
- added C36, C38, C43: 100nF, symbol RF_Board_Symbols:C
- added C37, C39, C45: 10uF, symbol RF_Board_Symbols:C
- added C40, C41, C42, C44: 12pF, symbol RF_Board_Symbols:C
- added J1, J3: Conn_Coaxial, symbol RF_Board_Symbols:Conn_Coaxial
- added J2, J4: Conn_01x07_Male, symbol RF_Board_Symbols:Conn_01x07_Male
- added J5, J6, J7: Conn_01x06_Female, symbol RF_Board_Symbols:Conn_01x06_Female
- added U13: RFM95PW, symbol RF_Board_Symbols:RFM95PW
- added Y2, Y3: Crystal, symbol RF_Board_Symbols:Crystal
- U1, U2: footprint RF_Board_Footprints:QFP50P900X900X160-48N -> QFP50P900X900X160-48N
Connections:
- net +5V: now also J2.6 (Pin_6), J4.6 (Pin_6), U13.12 (VCC)
- net GND: now also U1.7 (DVSS), U2.7 (DVSS), C36.2, C37.1, C38.2, C39.1, C40.1, C41.1, C42.1, C43.2, C44.1, C45.1, J1.2 (Ext), J2.7 (Pin_7), J3.2 (Ext), J4.7 (Pin_7), U13.15 (GND), U13.17 (PAD), U13.8 (GND)
- net at C24.2: now also J1.1 (In)
- net CC2500_SCLK: now reaches U3.1 (SCLK)
- net CC2500_SCLK: now also U2.14 (P4.5/UCB1CLK)
- net +3.3V: now reaches U3.11 (AVDD), U3.14 (AVDD), U3.15 (AVDD), U3.9 (AVDD)
- net +3.3V: now also U1.6 (DVCC), U2.6 (DVCC), U3.18 (VDD_GUARD), U3.4 (DVDD), C36.1, C37.2, C38.1, C39.2, C43.1, C45.2, J2.5 (Pin_5), J4.5 (Pin_5)
- net CC2500_MISO: now reaches U3.2 (SO(GDO1))
- net CC2500_MISO: now also U2.12 (P4.7/UCB1SOMI/UCB1SCL)
- net CC2500_MOSI: now reaches U3.20 (SI)
- net CC2500_MOSI: now also U2.13 (P4.6/UCB1SIMO/UCB1SDA)
- net GDO2: now reaches U3.3 (GDO2)
- net GDO2: now also U2.28 (P2.2/TB1CLK)
- net GDO0: now reaches U3.6 (GDO0(ATEST))
- net GDO0: now also U2.30 (P2.0/TB1.1/COMP0.O)
- net CC2500_CSN: now reaches U3.7 (~{CS})
- net CC2500_CSN: now also U2.15 (P4.4/UCB1STE)
- net RFM_MISO: now reaches U1.12 (P4.7/UCB1SOMI/UCB1SCL)
- net RFM_MISO: now also U13.2 (MISO)
- net RFM_MOSI: now reaches U1.13 (P4.6/UCB1SIMO/UCB1SDA)
- net RFM_MOSI: now also U13.3 (MOSI)
- net RFM_SCLK: now reaches U1.14 (P4.5/UCB1CLK)
- net RFM_SCLK: now also U13.4 (SCK)
- net RFM_CSN: now reaches U1.15 (P4.4/UCB1STE)
- net RFM_CSN: now also U13.5 (NSS)
- net RFM_UART_TX_2: now reaches U1.23 (P4.3/UCA1TXD/UCA1SIMO/~{UCA1TXD})
- net RFM_UART_TX_2: now also J4.3 (Pin_3)
- net RFM_UART_RX_2: now reaches U1.24 (P4.2/UCA1RXD/UCA1SOMI/~{UCA1RXD})
- net RFM_UART_RX_2: now also J4.4 (Pin_4)
- net RFM_UART_TX: now reaches U1.31 (P1.7/UCA0TXD/UCA0SIMO/TB0.2/TDO/OA1+/A7/VREF+)
- net RFM_UART_RX: now reaches U1.32 (P1.6/UCA0RXD/UCA0SOMI/TB0.1/TDI/TCLK/OA1-/A6)
- net RFM_SBWTCK: now reaches U1.4 (TEST/SBWTCK)
- net RFM_SBWTCK: now also J4.1 (Pin_1)
- net RFM_SBWTDIO: now reaches U1.5 (~{RST~{/NMI/SBWTDIO})
- net RFM_SBWTDIO: now also J4.2 (Pin_2)
- net RFM_XIN: now reaches U1.8 (P2.7/TB0CLK/XIN)
- net RFM_XIN: now also C42.2, Y3.1
- net RFM_XOUT: now reaches U1.9 (P2.6/MCLK/XOUT)
- net RFM_XOUT: now also C44.2, Y3.2
- net CC2500_UART_TX_2: now reaches U2.23 (P4.3/UCA1TXD/UCA1SIMO/~{UCA1TXD})
- net CC2500_UART_TX_2: now also J2.3 (Pin_3)
- net CC2500_UART_RX_2: now reaches U2.24 (P4.2/UCA1RXD/UCA1SOMI/~{UCA1RXD})
- net CC2500_UART_RX_2: now also J2.4 (Pin_4)
- net CC2500_UART_TX: now reaches U2.31 (P1.7/UCA0TXD/UCA0SIMO/TB0.2/TDO/OA1+/A7/VREF+)
- net CC2500_UART_RX: now reaches U2.32 (P1.6/UCA0RXD/UCA0SOMI/TB0.1/TDI/TCLK/OA1-/A6)
- net CC2500_SBWTCK: now reaches U2.4 (TEST/SBWTCK)
- net CC2500_SBWTCK: now also J2.1 (Pin_1)
- net CC2500_SBWTDIO: now reaches U2.5 (~{RST~{/NMI/SBWTDIO})
- net CC2500_SBWTDIO: now also J2.2 (Pin_2)
- net CC2500_XIN: now reaches U2.8 (P2.7/TB0CLK/XIN)
- net CC2500_XIN: now also C40.2, Y2.1
- net CC2500_XOUT: now reaches U2.9 (P2.6/MCLK/XOUT)
- net CC2500_XOUT: now also C41.2, Y2.2
- new net: J3.1 (In), U13.16 (ANT)
- new net RFM_RST: U13.6 (RESET)
Other:
- moved on the sheet: C1, C10, C11, C12, C13, C14, C15, C16, C17, C18, C19, C2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
