File: hardware/FlightComputer/FlightComputer.kicad_sch (KiCad schematic)
At the start: 75 parts, among them IC1 TPS54295PWPR, J1 Screw_Terminal_01x02, J2 SWD, J3 USB_B_Micro, J4 IMU, J5 Mag, J6 Camera, SW1 SW_SPDT, U1 SN74LVC2G04DCKR, U2 STM32F103VCT6, U3 LM75AD, U4 LM75AD, U5 LM75AD, U6 USBLC6-2SC6

Commit message: add breakouts
Parts:
- removed R5, R6: Resistor, symbol FCU-altium-import:3_Resistor
- removed U3, U4, U5: LM75AD, symbol LM75A:SO8
- added IC? (x3): LM75AD,118, SOIC127P600X175-8N, symbol SamacSys_Parts:LM75AD,118
- added J?: Conn_01x20_Male, symbol Connector:Conn_01x20_Male
- added J? (x2): Conn_01x20_Male, Connector_PinHeader_2.54mm:PinHeader_1x20_P2.54mm_Vertical, symbol Connector:Conn_01x20_Male
- added R5: 73.2k, symbol Device:R_Small
- added R6: 22.1k, symbol Device:R_Small
- added S?: 206-121S, 206121S, symbol SamacSys_Parts:206-121S
- gave numbers to parts that had none: 4
- renumbered J5 to J6, J6 to J7, R11 to R10, R12 to R11, R13 to R12, R14 to R13, R15 to R14, R16 to R15, R10 to R16, R8 to R7, R9 to R8, R7 to R9
Connections:
- net +3.3V: now also IC?.5 (A2), IC?.6 (A1), IC?.6 (A1), IC?.7 (A0), IC?.7 (A0), IC?.7 (A0), IC?.8 (VCC), IC?.8 (VCC), IC?.8 (VCC), J?.11 (Pin_11), J?.12 (Pin_12), J?.13 (Pin_13)
- net +3V3: now also R5.1
- net +5V: now also J?.14 (Pin_14), J?.15 (Pin_15)
- net ADC3_IN1: now also J?.17 (Pin_17)
- net ADC3_IN2: now also J?.18 (Pin_18)
- net ADC3_IN3: now also J?.19 (Pin_19)
- net DAC_OUT1: now also J?.20 (Pin_20)
- net GND: now also IC?.4 (GND), IC?.4 (GND), IC?.4 (GND), IC?.5 (A2), IC?.5 (A2), IC?.6 (A1), J?.10 (Pin_10), J?.18 (Pin_18), J?.3 (Pin_3), J?.4 (Pin_4), J?.5 (Pin_5), J?.6 (Pin_6), J?.7 (Pin_7), J?.8 (Pin_8), J?.9 (Pin_9)
- net GNDA: now also R6.2
- net I2C1_SCL: now also IC?.2 (SCL), IC?.2 (SCL), IC?.2 (SCL), J?.19 (Pin_19)
- net I2C1_SDA: now also IC?.1 (SDA), IC?.1 (SDA), IC?.1 (SDA), J?.20 (Pin_20)
- net PC15: now also J?.3 (Pin_3)
- net PC4: now also J?.17 (Pin_17)
- net PC5: now also J?.18 (Pin_18)
- net PC6: now also J?.19 (Pin_19)
- net PC7: now also J?.20 (Pin_20)
- net PC8: now also J?.1 (Pin_1)
- net PC9: now also J?.2 (Pin_2)
- net PD0: now also J?.1 (Pin_1)
- net PD1: now also J?.2 (Pin_2)
- net PD10: now also J?.11 (Pin_11)
- net PD11: now also J?.12 (Pin_12)
- net PD12: now also J?.13 (Pin_13)
- net PD13: now also J?.14 (Pin_14)
- net PD14: now also J?.15 (Pin_15)
- net PD15: now also J?.16 (Pin_16)
- net PD3: now also J?.4 (Pin_4)
- net PD4: now also J?.5 (Pin_5)
- net PD7: now also J?.8 (Pin_8)
- net PD8: now also J?.9 (Pin_9)
- net PD9: now also J?.10 (Pin_10)
- net PE0: now also J?.1 (Pin_1)
- net PE1: now also J?.2 (Pin_2)
- net PE10: now also J?.11 (Pin_11)
- net PE11: now also J?.12 (Pin_12)
- net PE12: now also J?.13 (Pin_13)
- net PE13: now also J?.14 (Pin_14)
- net PE14: now also J?.15 (Pin_15)
- net PE15: now also J?.16 (Pin_16)
- net PE2: now also J?.3 (Pin_3)
- net PE3: now also J?.4 (Pin_4)
- net PE4: now also J?.5 (Pin_5)
- net PE5: now also J?.6 (Pin_6)
- net PE6: now also J?.7 (Pin_7)
- net PE7: now also J?.8 (Pin_8)
- net PE8: now also J?.9 (Pin_9)
- net PE9: now also J?.10 (Pin_10)
- net VFB2: now also R5.2, R6.1
- net PD5 renamed UART2_TX
- net UART2_TX: now also J?.6 (Pin_6)
- net PD6 renamed UART2_RX
- net UART2_RX: now also J?.7 (Pin_7)
- net VIN renamed VDC
- net VDC: now also J?.16 (Pin_16), J?.17 (Pin_17)
Other:
- note added: "Breakout Headers"
- moved on the sheet: C23, C24, J6, J7, R16, Y1

Commit message: supposedly done with schematic
Parts:
- removed J?: Conn_01x20_Male, Connector_PinHeader_2.54mm:PinHeader_1x20_P2.54mm_Vertical, symbol Connector:Conn_01x20_Male
- removed R9: 10k, symbol Device:R_Small
- removed SW1: SW_SPDT, symbol Switch:SW_SPDT
- added J? (x2): Conn_01x20_Male, Connector_PinHeader_2.54mm:PinHeader_1x20_P2.54mm_Vertical, symbol Connector:Conn_01x20_Male
- added R7: 10k, symbol Device:R_Small
- gave numbers to parts that had none: 6
- renumbered R16 to R11, R11 to R12, R12 to R13, R13 to R14, R14 to R15, R15 to R16, R7 to R8, R8 to R9, U6 to U3
Connections:
- net +3.3V: now also J?.11 (Pin_11), J?.12 (Pin_12), J?.13 (Pin_13)
- net +3V3: now also S1.3 (COM_1)
- net +5V: now also J?.14 (Pin_14), J?.15 (Pin_15)
- net ADC3_IN10: now also J?.16 (Pin_16)
- net ADC3_IN11: now also J?.17 (Pin_17)
- net ADC3_IN12: now also J?.18 (Pin_18)
- net ADC3_IN13: now also J?.19 (Pin_19)
- net BOOT0: now also R7.1
- net GND: now also S1.4 (COM_2), J?.10 (Pin_10), J?.18 (Pin_18), J?.19 (Pin_19), J?.20 (Pin_20), J?.20 (Pin_20), J?.3 (Pin_3), J?.4 (Pin_4), J?.5 (Pin_5), J?.6 (Pin_6), J?.7 (Pin_7), J?.7 (Pin_7), J?.8 (Pin_8), J?.9 (Pin_9)
- net I2C1_SCL: now also J?.1 (Pin_1)
- net I2C1_SDA: now also J?.2 (Pin_2)
- net I2C2_SCL: now also J?.8 (Pin_8)
- net I2C2_SDA: now also J?.9 (Pin_9)
- net PC15: now also J?.3 (Pin_3)
- net PC8: now also J?.1 (Pin_1)
- net PC9: now also J?.2 (Pin_2)
- net SPI2_MISO: now also J?.5 (Pin_5)
- net SPI2_MOSI: now also J?.6 (Pin_6)
- net SPI2_SCK: now also J?.4 (Pin_4)
- net VDC: now also J?.16 (Pin_16), J?.17 (Pin_17)
- net at S1.1 (NO): now also R7.2
- no-connect marks 9 -> 11
Other:
- moved on the sheet: J2, S1

Commit message: Update FlightComputer.kicad_sch
Parts:
- gave numbers to parts that had none: 2
- renumbered J10 to J9
Connections:
- no-connect marks 11 -> 17
Other:
- moved on the sheet: J10, J11, J9

Commit message: update footprints
Parts:
- removed C5, C6: Capacitor 10nF +/-20% 50V 0402, CAPC0402(1005)60_L, symbol FCU-altium-import:0_CAP-NP-2
- removed S1: 206-121S, 206121S, symbol SamacSys_Parts:206-121S
- added C5, C6: 10u, Capacitor_SMD:C_1206_3216Metric_Pad1.33x1.80mm_HandSolder, symbol Device:C_Small
- added H1, H2, H3, H4: MountingHole_Pad, MountingHole:MountingHole_4.3mm_M4_Pad_Via, symbol Mechanical:MountingHole_Pad
- added J12: Boot Mode Select Headers, Connector_PinHeader_2.54mm:PinHeader_1x03_P2.54mm_Vertical, symbol Connector:Conn_01x03_Male
- C1, C12, C13, C14, C15, C16, C17, C18, C19, C2, C20, C21, C22, C23, C24, C3, C4, C7, C8, C9: footprint (none) -> Capacitor_SMD:C_0603_1608Metric_Pad1.08x0.95mm_HandSolder
- C10, C11: value Capacitor -> 22n; footprint (none) -> Capacitor_SMD:C_0603_1608Metric_Pad1.08x0.95mm_HandSolder
- D1: footprint (none) -> LED_SMD:LED_0603_1608Metric_Pad1.05x0.95mm_HandSolder
- IC2, IC3, IC4: footprint SOIC127P600X175-8N -> Package_SO:SOIC-8-1EP_3.9x4.9mm_P1.27mm_EP2.29x3mm_ThermalVias
- J1: footprint (none) -> TerminalBlock_Altech:Altech_AK300_1x02_P5.00mm_45-Degree
- J2: footprint (none) -> Connector_PinSocket_1.27mm:PinSocket_2x05_P1.27mm_Vertical_SMD
- J3: footprint (none) -> Connector_USB:USB_Micro-B_Molex_47346-0001
- J4: footprint (none) -> Connector_PinHeader_2.54mm:PinHeader_1x05_P2.54mm_Vertical
- J5: footprint L77TSAH15SOL2RM8 -> Connector_Dsub:DSUB-15_Female_Vertical_P2.77x2.84mm_MountingHoles
- J7: footprint (none) -> Connector_PinHeader_2.54mm:PinHeader_1x08_P2.54mm_Vertical
- J8: footprint (none) -> Connector_PinHeader_2.54mm:PinHeader_1x20_P2.54mm_Vertical
- L1, L2: footprint (none) -> Inductor_SMD:L_1812_4532Metric_Pad1.30x3.40mm_HandSolder
- L3: footprint (none) -> Inductor_SMD:L_01005_0402Metric_Pad0.57x0.30mm_HandSolder
- R1: value Resistor -> 124k; footprint (none) -> Resistor_SMD:R_0603_1608Metric_Pad0.98x0.95mm_HandSolder
- R10, R11, R12, R13, R14, R15, R16, R3, R4, R5, R6, R7, R8, R9: footprint (none) -> Resistor_SMD:R_0603_1608Metric_Pad0.98x0.95mm_HandSolder
- R2: value Resistor -> 22.1k; footprint (none) -> Resistor_SMD:R_0603_1608Metric_Pad0.98x0.95mm_HandSolder
- TP1, TP10, TP11, TP12, TP13, TP14, TP15, TP2, TP3, TP4, TP5, TP6, TP7, TP8, TP9: footprint (none) -> TestPoint:TestPoint_Keystone_5015_Micro-Minature
- U1: footprint FP-DCK0006A-IPC_B -> Package_SON:WSON-6_1.5x1.5mm_P0.5mm
- Y1: footprint ABM3B -> Crystal:Crystal_SMD_Abracon_ABM3B-4Pin_5.0x3.2mm
Connections:
- net +3V3: now also J12.1 (Pin_1)
- net GND: now also C5.2, C6.2, H1.1, H2.1, H3.1, H4.1, J12.3 (Pin_3)
- net VDC: now also C5.1, C6.1
- net at R7.2: now also J12.2 (Pin_2)
Other:
- moved on the sheet: C1, C11, C2, C8, J2, L1, L2, R7
