File: hardware/FlightComputer/FlightComputer.kicad_sch (KiCad schematic)
At the start: 83 parts, among them IC1 TPS54295PWPR, IC2 LM75AD,118, IC3 LM75AD,118, IC4 LM75AD,118, J1 Screw_Terminal_01x02, J10 Conn_01x20_Male, J11 Conn_01x20_Male, J12 Boot Mode Select Headers, J2 SWD, J3 USB_B_Micro, J4 IMU, J5 L77TSAH15SOL2RM8, J6 Mag, J7 Camera, J8 Conn_01x20_Male, J9 Conn_01x20_Male, U1 SN74LVC2G04DCKR, U2 STM32F103VCT6, U3 USBLC6-2SC6, Y1 ABM3B-8.000MHZ-10-1-U-T

Commit message: spaghetti
Parts:
- removed TP15: TestPoint, TestPoint:TestPoint_Keystone_5015_Micro-Minature, symbol Connector:TestPoint
- IC1: footprint C:_Users_Joey_Documents_AltiumLL_SamacSys.PcbLib_SOP65P640X120-17N -> Package_SO:HTSSOP-16-1EP_4.4x5mm_P0.65mm_EP3.4x5mm_Mask2.46x2.31mm_ThermalVias
- L1: value Inductor -> 3.3u
- L2: value Inductor -> 2.2u
- L3: footprint Inductor_SMD:L_01005_0402Metric_Pad0.57x0.30mm_HandSolder -> Inductor_SMD:L_0603_1608Metric_Pad1.05x0.95mm_HandSolder
- TP1: value TestPoint -> 5V
- TP10: value TestPoint -> I2C1_SCL
- TP11: value TestPoint -> I2C1_SDA
- TP12: value TestPoint -> I2C2_SCL
- TP13: value TestPoint -> I2C2_SDA
- TP14: value TestPoint -> GND
- TP2: value TestPoint -> EN1
- TP3: value TestPoint -> EN2
- TP4: value TestPoint -> 3V3
- TP5: value TestPoint -> SPI1_SCK
- TP6: value TestPoint -> SPI1_MISO
- TP7: value TestPoint -> SPI1_MOSI
- TP8: value TestPoint -> CS1
- TP9: value TestPoint -> CS2
Connections:
- net +3V3 is gone; now on net +3.3V: C10.1, C11.1, C14.1, C16.1, C18.1, C19.1, C20.1, C21.1, C22.1, J12.1 (Pin_1), J2.1 (Pin_1), L2.2, L3.1, R12.1, R13.1, R5.1, R8.1, R9.1, TP4.1, U2.100 (VDD), U2.11 (VDD), U2.28 (VDD), U2.50 (VDD), U2.6 (VBAT), U2.75 (VDD)
- net +5VD is gone; now on net +5V: J3.1 (VBUS), R14.1, U3.5 (VBUS)
- net GNDA is gone; now on net GND: C4.1, C8.2, R2.2, R6.2, U2.19 (VSSA)
- net ADC3_IN1: now also J8.8 (Pin_8); no longer J8.17 (Pin_17), U2.24 (PA1)
- net ADC3_IN10: no longer U2.15 (PC0)
- net ADC3_IN11: no longer U2.16 (PC1)
- net ADC3_IN12: no longer U2.17 (PC2)
- net ADC3_IN2: now also J8.9 (Pin_9); no longer J8.18 (Pin_18), U2.25 (PA2)
- net ADC3_IN3: now also J8.10 (Pin_10); no longer J8.19 (Pin_19), U2.26 (PA3)
- net DAC_OUT1: now also J8.11 (Pin_11); no longer J8.20 (Pin_20)
- net GND: now also J11.12 (Pin_12), J11.13 (Pin_13), J3.6 (Shield)
- net PC15: no longer U2.9 (PC15)
- net PC4: no longer J9.17 (Pin_17)
- net PD10: now also J9.14 (Pin_14); no longer J9.11 (Pin_11)
- net PD11: now also J9.13 (Pin_13); no longer J9.12 (Pin_12)
- net PD12: now also J9.12 (Pin_12); no longer J9.13 (Pin_13)
- net PD13: now also J9.11 (Pin_11); no longer J9.14 (Pin_14)
- net PD14: now also J9.10 (Pin_10); no longer J9.15 (Pin_15)
- net PD15: now also J9.9 (Pin_9); no longer J9.16 (Pin_16)
- net PD3: no longer U2.84 (PD3)
- net PD4: no longer U2.85 (PD4)
- net PD8: no longer J9.9 (Pin_9)
- net PD9: no longer J9.10 (Pin_10)
- net PE0: no longer U2.97 (PE0)
- net PE1: no longer U2.98 (PE1)
- net PE10: now also J8.15 (Pin_15); no longer J8.11 (Pin_11)
- net PE11: now also J8.16 (Pin_16); no longer J8.12 (Pin_12)
- net PE12: now also J8.17 (Pin_17); no longer J8.13 (Pin_13)
- net PE13: now also J8.18 (Pin_18); no longer J8.14 (Pin_14)
- net PE14: now also J8.19 (Pin_19); no longer J8.15 (Pin_15)
- net PE15: now also J8.20 (Pin_20); no longer J8.16 (Pin_16)
- net PE5: no longer U2.4 (PE5)
- net PE6: no longer U2.5 (PE6)
- net PE7: now also J8.12 (Pin_12); no longer J8.8 (Pin_8)
- net PE8: now also J8.13 (Pin_13); no longer J8.9 (Pin_9)
- net PE9: no longer J8.10 (Pin_10)
- net SPI2_MISO: now also J9.16 (Pin_16); no longer J11.5 (Pin_5)
- net SPI2_MOSI: now also J9.15 (Pin_15); no longer J11.6 (Pin_6)
- net SPI2_SCK: now also J9.17 (Pin_17); no longer J11.4 (Pin_4)
- net PC5: no longer names the net of J9.18 (Pin_18)
- net PC5: no longer U2.34 (PC5)
- net PC6: no longer names the net of J9.19 (Pin_19)
- net PC6: no longer U2.63 (PC6)
- net PC7: no longer names the net of J9.20 (Pin_20)
- net PC7: no longer U2.64 (PC7)
- net PD0: no longer names the net of J9.1 (Pin_1)
- net PD0: no longer U2.81 (PD0)
- net PD1: no longer names the net of J9.2 (Pin_2)
- net PD1: no longer U2.82 (PD1)
- no-connect marks 17 -> 41
