File: hardware/FlightComputer/FlightComputer.kicad_pcb (KiCad board)
At the start: 4 copper layers, 90 x 90 mm, 83 parts, among them IC1 TPS54295PWPR, IC2 LM75AD,118, IC3 LM75AD,118, IC4 LM75AD,118, J1 Screw_Terminal_01x02, J10 Conn_01x20_Male, J11 Conn_01x20_Male, J12 Boot Mode Select Headers, J2 SWD, J3 USB_B_Micro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

Commit message: slight change, output again
Routing:
- net PC9: track 30.9 -> 40.2 mm, vias 2 -> 1
- net PC8: track 36.1 -> 43.1 mm, vias 2 -> 0
- net I2C1_SDA: track 182.0 -> 181.2 mm
- net UART2_RX: track 32.6 -> 33.3 mm
- net SPI1_SCK: track 61.1 -> 61.6 mm
